File: tcu/$tcu.sch (KiCad schematic (older format))
At the start: 52 parts, among them CON1 USB-MICRO-B, K1 SPDT_RELAY, K2 SPDT_RELAY, K3 SPDT_RELAY, P1 CONN_01X08, P2 CONN_02X03, P3 NRF24L01+, P4 ESP8266, Q1 E_NMOS, Q2 E_NMOS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

Commit message: started routing
external connections mostly done
Parts:
- F1: footprint (none) -> SMD_Packages:SMD-0603
- L1: footprint (none) -> Inductor:SMD_Inductor
- Q1, Q2, Q3, Q4: footprint (none) -> SMD_Packages:SOT-23-GDS
Changed lines of the file:
@@
 F 0 "L1" V 6500 1050 40  0000 C CNN
 F 1 "22uH" V 6650 1050 40  0000 C CNN
-F 2 "" H 6550 1050 60  0001 C CNN
+F 2 "Inductor:SMD_Inductor" H 6550 1050 60  0001 C CNN
 F 3 "" H 6550 1050 60  0000 C CNN
 	1    6550 1050
@@
 F 0 "Q3" H 3660 1620 60  0000 R CNN
 F 1 "E_NMOS" H 3650 1300 60  0000 R CNN
-F 2 "" H 3650 1450 60  0001 C CNN
+F 2 "SMD_Packages:SOT-23-GDS" H 3650 1450 60  0001 C CNN
 F 3 "" H 3650 1450 60  0000 C CNN
 	1    3650 1450
@@
 F 0 "Q1" H 3610 2870 60  0000 R CNN
 F 1 "E_NMOS" H 3600 2550 60  0000 R CNN
-F 2 "" H 3600 2700 60  0001 C CNN
+F 2 "SMD_Packages:SOT-23-GDS" H 3600 2700 60  0001 C CNN
 F 3 "" H 3600 2700 60  0000 C CNN
 	1    3600 2700
@@
 F 0 "Q2" H 3610 4070 60  0000 R CNN
 F 1 "E_NMOS" H 3600 3750 60  0000 R CNN
-F 2 "" H 3600 3900 60  0001 C CNN
+F 2 "SMD_Packages:SOT-23-GDS" H 3600 3900 60  0001 C CNN
 F 3 "" H 3600 3900 60  0000 C CNN
 	1    3600 3900
@@
 F 0 "Q4" H 9910 1020 60  0000 R CNN
 F 1 "E_NMOS" H 9900 700 60  0000 R CNN
-F 2 "" H 9900 850 60  0001 C CNN
+F 2 "SMD_Packages:SOT-23-GDS" H 9900 850 60  0001 C CNN
 F 3 "" H 9900 850 60  0000 C CNN
 	1    9900 850
@@
 F 0 "F1" H 5100 2000 40  0000 C CNN
 F 1 "500mA" H 4900 1900 40  0000 C CNN
-F 2 "" H 5000 1950 60  0001 C CNN
+F 2 "SMD_Packages:SMD-0603" H 5000 1950 60  0001 C CNN
 F 3 "" H 5000 1950 60  0000 C CNN
 	1    5000 1950
