File: tcu/_autosave-tcu.kicad_pcb (KiCad board)
At the start: 2 copper layers, 52 parts, among them CON1 USB-MICRO-B, K1 SPDT_RELAY, K2 SPDT_RELAY, K3 SPDT_RELAY, P1 CONN_01X08, P2 CONN_02X03, P3 NRF24L01+, P4 ESP8266, Q1 E_NMOS, Q2 E_NMOS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

Commit message: started routing
external connections mostly done
Routing:
- net GND: track 0.00 -> 86.4 mm
- net Net-(BR2-Pad1): track 0.00 -> 59.3 mm
- net Net-(BR3-Pad2): track 0.00 -> 53.3 mm
- net Net-(BR3-Pad1): track 0.00 -> 36.8 mm
- net Net-(BR1-Pad1): track 0.00 -> 31.8 mm
- net Net-(BR1-Pad2): track 0.00 -> 27.9 mm
- net Net-(BR2-Pad2): track 18.9 -> 32.9 mm
- net Net-(D5-Pad2): track 0.00 -> 8.07 mm
- net Net-(D4-Pad2): track 0.00 -> 8.07 mm
- net Net-(K2-Pad5): track 0.00 -> 6.52 mm
- net Net-(K1-Pad5): track 0.00 -> 6.52 mm
- net Net-(BR2-Pad3): track 0.00 -> 5.61 mm
- net Net-(BR1-Pad3): track 0.00 -> 5.61 mm
Other:
- net class power added: clearance 0.254, trace_width 0.6096, via_dia 0.889, via_drill 0.635
Changed lines of the file:
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@@
     (thickness 1.6)
     (drawings 0)
-    (tracks 2)
+    (tracks 60)
     (zones 0)
     (modules 52)
@@
   )
   (setup
-    (last_trace_width 0.254)
+    (last_trace_width 0.6096)
+    (user_trace_width 0.3048)
+    (user_trace_width 0.6096)
     (trace_clearance 0.254)
     (zone_clearance 0.508)
@@
     (add_net /TEMPERATURE)
     (add_net /TXD)
-    (add_net /UVCC)
     (add_net /X+)
     (add_net /X-)
     (add_net /Y+)
     (add_net /Y-)
-    (add_net GND)
     (add_net "Net-(BR1-Pad1)")
     (add_net "Net-(BR1-Pad2)")
@@
     (add_net "Net-(U2-Pad22)")
     (add_net "Net-(U2-Pad30)")
+  )
+  (net_class power ""
+    (clearance 0.254)
+    (trace_width 0.6096)
+    (via_dia 0.889)
+    (via_drill 0.635)
+    (uvia_dia 0.508)
+    (uvia_drill 0.127)
+    (add_net /UVCC)
+    (add_net GND)
     (add_net VCC)
+  )
+  (module Relay:G5LE (layer F.Cu)
+    (at 38.1 -27.94 180)
+    (fp_text reference K2 (at 0 0 180) (layer F.SilkS)
+      (effects (font (size 1.5 1.5) (thickness 0.15)))
+    )
+    (fp_text value SPDT_RELAY (at 0 0 180) (layer F.SilkS)
+      (effects (font (size 1.5 1.5) (thickness 0.15)))
+    )
+    (fp_line (start -4.55 2.25) (end -4.55 -6) (layer F.SilkS) (width 0.15))
+    (fp_line (start 17.95 2.25) (end -4.55 2.25) (layer F.SilkS) (width 0.15))
+    (fp_line (start 17.95 -14.25) (end 17.95 2.25) (layer F.SilkS) (width 0.15))
+    (fp_line (start -4.55 -14.25) (end 17.95 -14.25) (layer F.SilkS) (width 0.15))
+    (fp_line (start -4.55 -6) (end -4.55 -14.25) (layer F.SilkS) (width 0.15))
+    (pad 5 thru_hole circle (at 0 0 180) (size 2.5 2.5) (drill 1.5) (layers *.Cu *.Mask F.SilkS)
+      (net 65 "Net-(K2-Pad5)"))
+    (pad 2 thru_hole circle (at 0 -12 180) (size 2.5 2.5) (drill 1.5) (layers *.Cu *.Mask F.SilkS)
+      (net 17 VCC))
+    (pad 3 thru_hole circle (at 12.2 -12 180) (size 2.5 2.5) (drill 1.5) (layers *.Cu *.Mask F.SilkS)
+      (net 5 "Net-(BR2-Pad1)"))
+    (pad 4 thru_hole circle (at 12.2 0 180) (size 2.5 2.5) (drill 1.5) (layers *.Cu *.Mask F.SilkS)
+      (net 66 "Net-(K2-Pad4)"))
+    (pad 1 thru_hole circle (at -2 -6 180) (size 2.5 2.5) (drill 1.5) (layers *.Cu *.Mask F.SilkS)
+      (net 6 "Net-(BR2-Pad2)"))
   )
   (module "Bridge Rectifiers:GBU4" (layer F.Cu)
@@
   )
   (module Relay:G5LE (layer F.Cu)
-    (at 38.1 -27.94 180)
-    (fp_text reference K2 (at 0 0 180) (layer F.SilkS)
-      (effects (font (size 1.5 1.5) (thickness 0.15)))
-    )
-    (fp_text value SPDT_RELAY (at 0 0 180) (layer F.SilkS)
-      (effects (font (size 1.5 1.5) (thickness 0.15)))
-    )
-    (fp_line (start -4.55 2.25) (end -4.55 -6) (layer F.SilkS) (width 0.15))
-    (fp_line (start 17.95 2.25) (end -4.55 2.25) (layer F.SilkS) (width 0.15))
-    (fp_line (start 17.95 -14.25) (end 17.95 2.25) (layer F.SilkS) (width 0.15))
-    (fp_line (start -4.55 -14.25) (end 17.95 -14.25) (layer F.SilkS) (width 0.15))
-    (fp_line (start -4.55 -6) (end -4.55 -14.25) (layer F.SilkS) (width 0.15))
-    (pad 5 thru_hole circle (at 0 0 180) (size 2.5 2.5) (drill 1.5) (layers *.Cu *.Mask F.SilkS)
-      (net 65 "Net-(K2-Pad5)"))
-    (pad 2 thru_hole circle (at 0 -12 180) (size 2.5 2.5) (drill 1.5) (layers *.Cu *.Mask F.SilkS)
-      (net 17 VCC))
-    (pad 3 thru_hole circle (at 12.2 -12 180) (size 2.5 2.5) (drill 1.5) (layers *.Cu *.Mask F.SilkS)
-      (net 5 "Net-(BR2-Pad1)"))
-    (pad 4 thru_hole circle (at 12.2 0 180) (size 2.5 2.5) (drill 1.5) (layers *.Cu *.Mask F.SilkS)
-      (net 66 "Net-(K2-Pad4)"))
-    (pad 1 thru_hole circle (at -2 -6 180) (size 2.5 2.5) (drill 1.5) (layers *.Cu *.Mask F.SilkS)
-      (net 6 "Net-(BR2-Pad2)"))
-  )
-  (module Relay:G5LE (layer F.Cu)
     (at 99.06 -27.94 180)
     (fp_text reference K3 (at 0 0 180) (layer F.SilkS)
@@
     (tags "CMS SOT")
     (attr smd)
-    (fp_text reference Q4 (at 0 -2.159) (layer F.SilkS)
+    (fp_text reference Q4 (at 0 -2.54) (layer F.SilkS)
       (effects (font (size 1 1) (thickness 0.15)))
     )
@@
       (net 15 "Net-(C5-Pad1)"))
   )
-  (segment (start 41.91 -41.91) (end 48.26 -41.91) (width 0.254) (layer F.Cu) (net 6))
-  (segment (start 33.02 -33.02) (end 41.91 -41.91) (width 0.254) (layer F.Cu) (net 6))
+  (segment (start 58.42 -33.02) (end 58.42 -17.98) (width 0.6096) (layer B.Cu) (net 1))
+  (segment (start 58.42 -17.98) (end 56.38 -15.94) (width 0.6096) (layer B.Cu) (net 1))
+  (segment (start 58.42 -33.02) (end 67.31 -41.91) (width 0.6096) (layer F.Cu) (net 1))
+  (segment (start 67.31 -41.91) (end 68.58 -41.91) (width 0.6096) (layer F.Cu) (net 1))
+  (segment (start 63.5 -33.02) (end 63.5 -29.02) (width 0.6096) (layer B.Cu) (net 2))
+  (segment (start 63.5 -29.02) (end 70.58 -21.94) (width 0.6096) (layer B.Cu) (net 2))
+  (segment (start 63.5 -33.02) (end 54.61 -41.91) (width 0.6096) (layer B.Cu) (net 2))
+  (segment (start 54.61 -41.91) (end 53.34 -41.91) (width 0.6096) (layer B.Cu) (net 2))
+  (segment (start 68.58 -33.02) (end 74.1934 -33.02) (width 0.6096) (layer F.Cu) (net 3))
+  (segment (start 83.82 -33.02) (end 85.25684 -33.02) (width 0.6096) (layer F.Cu) (net 4))
+  (segment (start 85.25684 -33.02) (end 87.79684 -30.48) (width 0.6096) (layer F.Cu) (net 4))
+  (segment (start 87.79684 -30.48) (end 92.71 -30.48) (width 0.6096) (layer F.Cu) (net 4))
+  (segment (start 92.71 -30.48) (end 98.679 -24.511) (width 0.6096) (layer F.Cu) (net 4))
+  (segment (start 98.679 -24.511) (end 105.664 -24.511) (width 0.6096) (layer F.Cu) (net 4))
+  (segment (start 104.5972 -24.511) (end 105.664 -24.511) (width 0.6096) (layer F.Cu) (net 4))
+  (segment (start 62.23 -30.48) (end 68.199 -24.511) (width 0.6096) (layer F.Cu) (net 4))
+  (segment (start 68.199 -24.511) (end 75.184 -24.511) (width 0.6096) (layer F.Cu) (net 4))
+  (segment (start 57.31684 -30.48) (end 62.23 -30.48) (width 0.6096) (layer F.Cu) (net 4))
+  (segment (start 53.34 -33.02) (end 54.77684 -33.02) (width 0.6096) (layer F.Cu) (net 4))
+  (segment (start 54.77684 -33.02) (end 57.31684 -30.48) (width 0.6096) (layer F.Cu) (net 4))
+  (segment (start 31.75 -30.48) (end 37.719 -24.511) (width 0.6096) (layer F.Cu) (net 4))
+  (segment (start 37.719 -24.511) (end 44.704 -24.511) (width 0.6096) (layer F.Cu) (net 4))
+  (segment (start 25.4 -30.48) (end 31.75 -30.48) (width 0.6096) (layer F.Cu) (net 4))
+  (segment (start 22.86 -33.02) (end 25.4 -30.48) (width 0.6096) (layer F.Cu) (net 4))
+  (segment (start 75.184 -24.511) (end 75.184 -21.3106) (width 0.6096) (layer F.Cu) (net 4))
+  (segment (start 75.184 -21.3106) (end 74.1934 -20.32) (width 0.6096) (layer F.Cu) (net 4))
+  (segment (start 44.704 -24.511) (end 44.704 -21.3106) (width 0.6096) (layer F.Cu) (net 4))
+  (segment (start 44.704 -21.3106) (end 43.7134 -20.32) (width 0.6096) (layer F.Cu) (net 4))
+  (segment (start 27.94 -33.02) (end 27.94 -17.98) (width 0.6096) (layer B.Cu) (net 5))
+  (segment (start 27.94 -17.98) (end 25.9 -15.94) (width 0.6096) (layer B.Cu) (net 5))
+  (segment (start 27.94 -33.02) (end 39.37 -44.45) (width 0.6096) (layer F.Cu) (net 5))
+  (segment (start 39.37 -44.45) (end 60.96 -44.45) (width 0.6096) (layer F.Cu) (net 5))
+  (segment (start 60.96 -44.45) (end 62.484001 -42.925999) (width 0.6096) (layer F.Cu) (net 5))
+  (segment (start 62.484001 -42.925999) (end 63.5 -41.91) (width 0.6096) (layer F.Cu) (net 5))
+  (segment (start 33.02 -33.02) (end 33.02 -29.02) (width 0.6096) (layer B.Cu) (net 6))
+  (segment (start 33.02 -29.02) (end 40.1 -21.94) (width 0.6096) (layer B.Cu) (net 6))
+  (segment (start 33.02 -33.02) (end 41.91 -41.91) (width 0.6096) (layer F.Cu) (net 6))
+  (segment (start 41.91 -41.91) (end 48.26 -41.91) (width 0.6096) (layer F.Cu) (net 6))
+  (segment (start 38.1 -33.02) (end 43.7134 -33.02) (width 0.6096) (layer F.Cu) (net 7))
+  (segment (start 88.9 -33.02) (end 88.9 -17.98) (width 0.6096) (layer B.Cu) (net 8))
+  (segment (start 88.9 -17.98) (end 86.86 -15.94) (width 0.6096) (layer B.Cu) (net 8))
+  (segment (start 88.9 -33.02) (end 85.09 -36.83) (width 0.6096) (layer F.Cu) (net 8))
+  (segment (start 85.09 -36.83) (end 78.74 -36.83) (width 0.6096) (layer F.Cu) (net 8))
+  (segment (start 78.74 -36.83) (end 73.66 -41.91) (width 0.6096) (layer F.Cu) (net 8))
+  (segment (start 93.98 -33.02) (end 93.98 -29.02) (width 0.6096) (layer B.Cu) (net 9))
+  (segment (start 93.98 -29.02) (end 101.06 -21.94) (width 0.6096) (layer B.Cu) (net 9))
+  (segment (start 93.98 -33.02) (end 90.17 -36.83) (width 0.6096) (layer B.Cu) (net 9))
+  (segment (start 90.17 -36.83) (end 63.5 -36.83) (width 0.6096) (layer B.Cu) (net 9))
+  (segment (start 63.5 -36.83) (end 59.435999 -40.894001) (width 0.6096) (layer B.Cu) (net 9))
+  (segment (start 59.435999 -40.894001) (end 58.42 -41.91) (width 0.6096) (layer B.Cu) (net 9))
+  (segment (start 77.216 -25.4) (end 77.216 -21.3106) (width 0.6096) (layer F.Cu) (net 21))
+  (segment (start 77.216 -21.3106) (end 78.2066 -20.32) (width 0.6096) (layer F.Cu) (net 21))
+  (segment (start 77.3 -27.94) (end 77.3 -25.484) (width 0.6096) (layer F.Cu) (net 21))
+  (segment (start 77.3 -25.484) (end 77.216 -25.4) (width 0.6096) (layer F.Cu) (net 21))
+  (segment (start 46.736 -25.4) (end 46.736 -21.3106) (width 0.6096) (layer F.Cu) (net 22))
+  (segment (start 46.736 -21.3106) (end 47.7266 -20.32) (width 0.6096) (layer F.Cu) (net 22))
+  (segment (start 46.82 -27.94) (end 46.82 -25.484) (width 0.6096) (layer F.Cu) (net 22))
+  (segment (start 46.82 -25.484) (end 46.736 -25.4) (width 0.6096) (layer F.Cu) (net 22))
+  (segment (start 68.58 -27.94) (end 75.1 -27.94) (width 0.6096) (layer F.Cu) (net 63))
+  (segment (start 38.1 -27.94) (end 44.62 -27.94) (width 0.6096) (layer F.Cu) (net 65))
 )
