File: tcu/tcu.sch (KiCad schematic (older format))
At the start: 52 parts, among them CON1 USB-MICRO-B, K1 SPDT_RELAY, K2 SPDT_RELAY, K3 SPDT_RELAY, P1 CONN_01X08, P2 CONN_02X03, P3 NRF24L01+, P4 ESP8266, Q1 E_NMOS, Q2 E_NMOS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

Commit message: assigned footprints
d1-d8, U1,t1,
Parts:
- P2: footprint (none) -> Pin_Headers:Pin_Header_Straight_2x03
- P4: footprint (none) -> Wireless modules:ESP8266
- VR1: footprint Crystals:Crystal_HC49-U_Vertical -> SMD_Packages:TO-263-5_HandSoldering
Connections:
- no-connect marks 33 -> 34
Changed lines of the file:
@@
 F 0 "P2" H 1600 5850 50  0000 C CNN
 F 1 "CONN_02X03" H 1600 5450 50  0000 C CNN
-F 2 "" H 1600 4450 60  0001 C CNN
+F 2 "Pin_Headers:Pin_Header_Straight_2x03" H 1600 4450 60  0001 C CNN
 F 3 "" H 1600 4450 60  0000 C CNN
 	1    1600 5650
@@
 F 0 "P4" H 1600 7400 50  0000 C CNN
 F 1 "ESP8266" H 1600 6900 50  0000 C CNN
-F 2 "" H 1600 5950 60  0001 C CNN
+F 2 "Wireless modules:ESP8266" H 1600 5950 60  0001 C CNN
 F 3 "" H 1600 5950 60  0000 C CNN
 	1    1600 7150
@@
 F 0 "VR1" H 4850 800 60  0000 C CNN
 F 1 "AP3003-3.3V" H 4900 1350 60  0000 C CNN
-F 2 "Crystals:Crystal_HC49-U_Vertical" H 5250 1050 60  0001 C CNN
+F 2 "SMD_Packages:TO-263-5_HandSoldering" H 5250 1050 60  0001 C CNN
 F 3 "" H 5250 1050 60  0000 C CNN
 	1    5300 1050
@@
 $EndComp
 $Comp
-L LM335 T1
-U 1 1 54B973A1
-P 3150 7400
-F 0 "T1" H 3300 7350 60  0000 C CNN
-F 1 "LM335" H 3400 7450 60  0000 C CNN
-F 2 "" H 3150 7400 60  0001 C CNN
-F 3 "" H 3150 7400 60  0000 C CNN
-	1    3150 7400
-	1    0    0    -1
-$EndComp
-$Comp
 L GND #PWR030
 U 1 1 54B99746
@@
 	1    0    0    -1
 $EndComp
+$Comp
+L LM335 T1
+U 1 1 54C8167B
+P 3150 7400
+F 0 "T1" H 3300 7350 60  0000 C CNN
+F 1 "LM335" H 3400 7450 60  0000 C CNN
+F 2 "" H 3150 7400 60  0000 C CNN
+F 3 "" H 3150 7400 60  0000 C CNN
+	1    3150 7400
+	1    0    0    -1
+$EndComp
+NoConn ~ 2850 7450
 $EndSCHEMATC

Commit message: created and assigned display connector footprint
Parts:
- D1, D2, D3, D4, D5, D6, D7, D8: footprint (none) -> SMD_Packages:DO-214-AA_SMB
- T1: footprint (none) -> Housings_TO-92:TO-92-Free-molded-wide
- U1: footprint (none) -> SMD_Packages:SOIC-8-W
Changed lines of the file:
@@
 F 0 "D1" H 3400 850 40  0000 C CNN
 F 1 "1N5822" H 3400 650 40  0000 C CNN
-F 2 "" H 3400 750 60  0001 C CNN
+F 2 "SMD_Packages:DO-214-AA_SMB" H 3400 750 60  0001 C CNN
 F 3 "" H 3400 750 60  0000 C CNN
 	1    3400 750
@@
 F 0 "D2" H 3400 2050 40  0000 C CNN
 F 1 "1N5822" H 3400 1850 40  0000 C CNN
-F 2 "" H 3400 1950 60  0001 C CNN
+F 2 "SMD_Packages:DO-214-AA_SMB" H 3400 1950 60  0001 C CNN
 F 3 "" H 3400 1950 60  0000 C CNN
 	1    3400 1950
@@
 F 0 "D3" H 3400 3300 40  0000 C CNN
 F 1 "1N5822" H 3400 3100 40  0000 C CNN
-F 2 "" H 3400 3200 60  0001 C CNN
+F 2 "SMD_Packages:DO-214-AA_SMB" H 3400 3200 60  0001 C CNN
 F 3 "" H 3400 3200 60  0000 C CNN
 	1    3400 3200
@@
 F 0 "D7" H 4450 2050 40  0000 C CNN
 F 1 "1N5822" H 4450 1850 40  0000 C CNN
-F 2 "" H 4450 1950 60  0001 C CNN
+F 2 "SMD_Packages:DO-214-AA_SMB" H 4450 1950 60  0001 C CNN
 F 3 "" H 4450 1950 60  0000 C CNN
 	1    4450 1950
@@
 F 0 "D4" H 3600 3050 40  0000 C CNN
 F 1 "1N5822" H 3600 2850 40  0000 C CNN
-F 2 "" H 3600 2950 60  0001 C CNN
+F 2 "SMD_Packages:DO-214-AA_SMB" H 3600 2950 60  0001 C CNN
 F 3 "" H 3600 2950 60  0000 C CNN
 	1    3600 2950
@@
 F 0 "D6" H 3650 1800 40  0000 C CNN
 F 1 "1N5822" H 3650 1600 40  0000 C CNN
-F 2 "" H 3650 1700 60  0001 C CNN
+F 2 "SMD_Packages:DO-214-AA_SMB" H 3650 1700 60  0001 C CNN
 F 3 "" H 3650 1700 60  0000 C CNN
 	1    3650 1700
@@
 F 0 "D5" H 3600 4250 40  0000 C CNN
 F 1 "1N5822" H 3600 4050 40  0000 C CNN
-F 2 "" H 3600 4150 60  0001 C CNN
+F 2 "SMD_Packages:DO-214-AA_SMB" H 3600 4150 60  0001 C CNN
 F 3 "" H 3600 4150 60  0000 C CNN
 	1    3600 4150
@@
 F 0 "U1" H 5550 6550 60  0000 L CNN
 F 1 "LM358" H 5550 6100 60  0000 L CNN
-F 2 "" H 5600 6350 60  0001 C CNN
+F 2 "SMD_Packages:SOIC-8-W" H 5600 6350 60  0001 C CNN
 F 3 "" H 5600 6350 60  0000 C CNN
 	2    5600 6350
@@
 F 0 "U1" H 3850 6000 60  0000 L CNN
 F 1 "LM358" H 3850 5550 60  0000 L CNN
-F 2 "" H 3900 5800 60  0001 C CNN
+F 2 "SMD_Packages:SOIC-8-W" H 3900 5800 60  0001 C CNN
 F 3 "" H 3900 5800 60  0000 C CNN
 	1    3900 5800
@@
 F 0 "D8" H 6150 1400 40  0000 C CNN
 F 1 "1N5822" H 6150 1200 40  0000 C CNN
-F 2 "" H 6150 1300 60  0001 C CNN
+F 2 "SMD_Packages:DO-214-AA_SMB" H 6150 1300 60  0001 C CNN
 F 3 "" H 6150 1300 60  0000 C CNN
 	1    6150 1300
@@
 F 0 "T1" H 3300 7350 60  0000 C CNN
 F 1 "LM335" H 3400 7450 60  0000 C CNN
-F 2 "" H 3150 7400 60  0000 C CNN
+F 2 "Housings_TO-92:TO-92-Free-molded-wide" H 3150 7400 60  0001 C CNN
 F 3 "" H 3150 7400 60  0000 C CNN
 	1    3150 7400

Commit message: further work on layout
Parts:
- D10: footprint (none) -> FPC Connector:FPC CONNECTOR
- F1: footprint (none) -> SMD_Packages:SMD-0603
- L1: footprint (none) -> Inductor:SMD_Inductor
- Q1, Q2, Q3, Q4: footprint (none) -> SMD_Packages:SOT-23-GDS
Changed lines of the file:
@@
 F 0 "L1" V 6500 1050 40  0000 C CNN
 F 1 "22uH" V 6650 1050 40  0000 C CNN
-F 2 "" H 6550 1050 60  0001 C CNN
+F 2 "Inductor:SMD_Inductor" H 6550 1050 60  0001 C CNN
 F 3 "" H 6550 1050 60  0000 C CNN
 	1    6550 1050
@@
 F 0 "D10" H 10550 750 60  0000 C CNN
 F 1 "MI0283QT-11" H 10800 5850 60  0000 C CNN
-F 2 "" H 10600 3350 60  0001 C CNN
+F 2 "FPC Connector:FPC CONNECTOR" H 10600 3350 60  0001 C CNN
 F 3 "" H 10600 3350 60  0000 C CNN
 	1    10800 3350
@@
 F 0 "Q3" H 3660 1620 60  0000 R CNN
 F 1 "E_NMOS" H 3650 1300 60  0000 R CNN
-F 2 "" H 3650 1450 60  0001 C CNN
+F 2 "SMD_Packages:SOT-23-GDS" H 3650 1450 60  0001 C CNN
 F 3 "" H 3650 1450 60  0000 C CNN
 	1    3650 1450
@@
 F 0 "Q1" H 3610 2870 60  0000 R CNN
 F 1 "E_NMOS" H 3600 2550 60  0000 R CNN
-F 2 "" H 3600 2700 60  0001 C CNN
+F 2 "SMD_Packages:SOT-23-GDS" H 3600 2700 60  0001 C CNN
 F 3 "" H 3600 2700 60  0000 C CNN
 	1    3600 2700
@@
 F 0 "Q2" H 3610 4070 60  0000 R CNN
 F 1 "E_NMOS" H 3600 3750 60  0000 R CNN
-F 2 "" H 3600 3900 60  0001 C CNN
+F 2 "SMD_Packages:SOT-23-GDS" H 3600 3900 60  0001 C CNN
 F 3 "" H 3600 3900 60  0000 C CNN
 	1    3600 3900
@@
 F 0 "Q4" H 9910 1020 60  0000 R CNN
 F 1 "E_NMOS" H 9900 700 60  0000 R CNN
-F 2 "" H 9900 850 60  0001 C CNN
+F 2 "SMD_Packages:SOT-23-GDS" H 9900 850 60  0001 C CNN
 F 3 "" H 9900 850 60  0000 C CNN
 	1    9900 850
@@
 F 0 "F1" H 5100 2000 40  0000 C CNN
 F 1 "500mA" H 4900 1900 40  0000 C CNN
-F 2 "" H 5000 1950 60  0001 C CNN
+F 2 "SMD_Packages:SMD-0603" H 5000 1950 60  0001 C CNN
 F 3 "" H 5000 1950 60  0000 C CNN
 	1    5000 1950
