File: TCU_HARDWARE/tcu.sch (KiCad schematic (older format))
At the start: 52 parts, among them CON1 USB-MICRO-B, K1 SPDT_RELAY, K2 SPDT_RELAY, K3 SPDT_RELAY, P1 CONN_01X08, P2 CONN_02X03, P3 NRF24L01+, P4 ESP8266, Q1 E_NMOS, Q2 E_NMOS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

Commit message: added pin definitions
Parts:
- R6: value 22 -> 10k
- R7: value 22 -> 52.3k
- R8: value 22 -> 1.8K
Changed lines of the file:
@@
 P 3150 5400
 F 0 "R6" V 3230 5400 40  0000 C CNN
-F 1 "22" V 3157 5401 40  0000 C CNN
+F 1 "10k" V 3157 5401 40  0000 C CNN
 F 2 "Resistors_SMD:R_0603_HandSoldering" V 3080 5400 30  0001 C CNN
 F 3 "" H 3150 5400 30  0000 C CNN
@@
 P 3150 6000
 F 0 "R7" V 3230 6000 40  0000 C CNN
-F 1 "22" V 3157 6001 40  0000 C CNN
+F 1 "52.3k" V 3157 6001 40  0000 C CNN
 F 2 "Resistors_SMD:R_0603_HandSoldering" V 3080 6000 30  0001 C CNN
 F 3 "" H 3150 6000 30  0000 C CNN
@@
 P 3150 6800
 F 0 "R8" V 3230 6800 40  0000 C CNN
-F 1 "22" V 3157 6801 40  0000 C CNN
+F 1 "1.8K" V 3157 6801 40  0000 C CNN
 F 2 "Resistors_SMD:R_0603_HandSoldering" V 3080 6800 30  0001 C CNN
 F 3 "" H 3150 6800 30  0000 C CNN
